File: BLDC-Control (1).kicad_sch (KiCad schematic)
At the start: 29 parts, among them J1 Screw_Terminal_01x08, J5 +24V Power, J6 +3V3 Power, Q1 Q_NMOS_GDS, Q2 Q_NMOS_GDS, Q3 Q_NMOS_GDS, Q4 Q_NMOS_GDS, Q5 Q_NMOS_GDS, Q6 Q_NMOS_GDS, U1 ESP32-WROOM-32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

Commit message: Add files via upload
changed SDATAI label on MCU to SDATAO to reflect MOSI pin
Connections:
- net SDATAI: no longer U1.37 (IO23)
- net SDATAO: now also U1.37 (IO23)
Changed lines of the file:
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@@
 		)
 	)
-	(label "SDATAI"
+	(label "SDATAO"
 		(at 76.2 153.67 0)
 		(effects
